File: NodeMCU/matriz.sch (KiCad schematic (older format))
At the start: 16 parts, among them J1 Conn_01x05, Q1 Q_NPN_CBE, Q2 Q_NPN_CBE, Q3 Q_NPN_CBE, SW1 SW_Push_Open, SW2 SW_Push, U3 NodeMCU1.0(ESP-12E)

Commit message: Avances entre todos
Parts:
- R1, R3, R5: value 50KOhm -> 500Ohm
- R2, R6: value 0.7KOhm -> 1000KOhm
- R4: value 0.7KOhm -> 1000Ohm
Other:
- moved on the sheet: Q1, R1, R2
Changed lines of the file:
@@
 L PWR_FLAG #FLG03
 U 1 1 5A09C060
-P 7800 6100
-F 0 "#FLG03" H 7800 6175 50  0001 C CNN
-F 1 "PWR_FLAG" H 7800 6250 50  0000 C CNN
-F 2 "" H 7800 6100 50  0001 C CNN
-F 3 "" H 7800 6100 50  0001 C CNN
-	1    7800 6100
+P 7850 6100
+F 0 "#FLG03" H 7850 6175 50  0001 C CNN
+F 1 "PWR_FLAG" H 7850 6250 50  0000 C CNN
+F 2 "" H 7850 6100 50  0001 C CNN
+F 3 "" H 7850 6100 50  0001 C CNN
+	1    7850 6100
 	1    0    0    -1
 $EndComp
@@
 L R R1
 U 1 1 5A048190
-P 7100 5000
-F 0 "R1" V 7200 5000 50  0000 C CNN
-F 1 "50KOhm" V 7300 5000 50  0000 C CNN
-F 2 "Resistors_THT:R_Axial_DIN0207_L6.3mm_D2.5mm_P7.62mm_Horizontal" V 7030 5000 50  0001 C CNN
-F 3 "" H 7100 5000 50  0001 C CNN
-	1    7100 5000
+P 7150 5100
+F 0 "R1" V 7250 5100 50  0000 C CNN
+F 1 "500Ohm" V 7350 5100 50  0000 C CNN
+F 2 "Resistors_THT:R_Axial_DIN0207_L6.3mm_D2.5mm_P7.62mm_Horizontal" V 7080 5100 50  0001 C CNN
+F 3 "" H 7150 5100 50  0001 C CNN
+	1    7150 5100
 	0    1    1    0
 $EndComp
@@
 L R R2
 U 1 1 5A048139
-P 7550 4550
-F 0 "R2" V 7630 4550 50  0000 C CNN
-F 1 "0.7KOhm" V 7700 4550 50  0000 C CNN
-F 2 "Resistors_THT:R_Axial_DIN0207_L6.3mm_D2.5mm_P7.62mm_Horizontal" V 7480 4550 50  0001 C CNN
-F 3 "" H 7550 4550 50  0001 C CNN
-	1    7550 4550
+P 7600 4650
+F 0 "R2" V 7680 4650 50  0000 C CNN
+F 1 "1000KOhm" V 7750 4650 50  0000 C CNN
+F 2 "Resistors_THT:R_Axial_DIN0207_L6.3mm_D2.5mm_P7.62mm_Horizontal" V 7530 4650 50  0001 C CNN
+F 3 "" H 7600 4650 50  0001 C CNN
+	1    7600 4650
 	-1   0    0    1
 $EndComp
@@
 P 8450 5150
 F 0 "R3" V 8550 5150 50  0000 C CNN
-F 1 "50KOhm" V 8650 5150 50  0000 C CNN
+F 1 "500Ohm" V 8650 5150 50  0000 C CNN
 F 2 "Resistors_THT:R_Axial_DIN0207_L6.3mm_D2.5mm_P7.62mm_Horizontal" V 8380 5150 50  0001 C CNN
 F 3 "" H 8450 5150 50  0001 C CNN
@@
 P 8900 4550
 F 0 "R4" V 8980 4550 50  0000 C CNN
-F 1 "0.7KOhm" V 9050 4550 50  0000 C CNN
+F 1 "1000Ohm" V 9050 4550 50  0000 C CNN
 F 2 "Resistors_THT:R_Axial_DIN0207_L6.3mm_D2.5mm_P7.62mm_Horizontal" V 8830 4550 50  0001 C CNN
 F 3 "" H 8900 4550 50  0001 C CNN
@@
 L GNDPWR #PWR04
 U 1 1 5A09BA2F
-P 7550 6200
-F 0 "#PWR04" H 7550 6000 50  0001 C CNN
-F 1 "GNDPWR" H 7550 6070 50  0000 C CNN
-F 2 "" H 7550 6150 50  0001 C CNN
-F 3 "" H 7550 6150 50  0001 C CNN
-	1    7550 6200
+P 7600 6200
+F 0 "#PWR04" H 7600 6000 50  0001 C CNN
+F 1 "GNDPWR" H 7600 6070 50  0000 C CNN
+F 2 "" H 7600 6150 50  0001 C CNN
+F 3 "" H 7600 6150 50  0001 C CNN
+	1    7600 6200
 	1    0    0    -1
 $EndComp
@@
 P 6800 3850
 F 0 "R5" V 6900 3850 50  0000 C CNN
-F 1 "50KOhm" V 7000 3850 50  0000 C CNN
+F 1 "500Ohm" V 7000 3850 50  0000 C CNN
 F 2 "Resistors_THT:R_Axial_DIN0207_L6.3mm_D2.5mm_P7.62mm_Horizontal" V 6730 3850 50  0001 C CNN
 F 3 "" H 6800 3850 50  0001 C CNN
@@
 P 7250 3250
 F 0 "R6" V 7330 3250 50  0000 C CNN
-F 1 "0.7KOhm" V 7400 3250 50  0000 C CNN
+F 1 "1000KOhm" V 7400 3250 50  0000 C CNN
 F 2 "Resistors_THT:R_Axial_DIN0207_L6.3mm_D2.5mm_P7.62mm_Horizontal" V 7180 3250 50  0001 C CNN
 F 3 "" H 7250 3250 50  0001 C CNN
@@
 	-1   0    0    1
 $EndComp
-Wire Wire Line
-	3800 2650 3800 2850
-Wire Wire Line
-	7900 2850 8850 2850
-Wire Wire Line
-	8400 3150 8850 3150
-Wire Wire Line
-	4100 2950 8850 2950
-Wire Wire Line
-	9650 5600 9650 2500
-Wire Wire Line
-	9650 2500 8350 2500
-Wire Wire Line
-	8350 2750 8850 2750
-Wire Wire Line
-	6600 5600 6600 5750
-Wire Wire Line
-	6350 5600 6350 5850
-Wire Wire Line
-	6100 5600 6100 5950
-Wire Wire Line
-	6600 4900 6600 5400
-Wire Wire Line
-	6100 5100 6100 5400
-Wire Wire Line
-	6350 5000 6350 5400
-Wire Wire Line
-	3800 2750 3500 2750
-Wire Wire Line
-	3500 2750 3500 2650
-Connection ~ 3800 2750
-Wire Wire Line
-	8350 2500 8350 2750
-Wire Wire Line
-	8150 3050 8850 3050
-Wire Wire Line
-	6950 4700 6100 4700
-Wire Wire Line
-	6100 4700 6100 4500
-Wire Wire Line
-	6100 4500 5750 4500
-Wire Wire Line
-	7550 5200 7550 6200
-Wire Wire Line
-	6100 5950 7550 5950
-Connection ~ 7550 5950
-Wire Wire Line
-	6350 5850 7550 5850
-Wire Wire Line
-	6600 5750 7550 5750
-Connection ~ 7550 5850
-Connection ~ 7550 5750
-Wire Wire Line
-	7550 6150 7800 6150
-Wire Wire Line
-	7800 6150 7800 6100
-Connection ~ 7550 6150
-Wire Wire Line
-	9400 3350 8400 3350
-Wire Wire Line
-	8400 3350 8400 3150
-Wire Wire Line
-	7550 5450 8900 5450
-Connection ~ 7550 5450
-Wire Wire Line
-	6500 4300 5750 4300
-Wire Wire Line
-	7250 4100 9650 4100
-Connection ~ 9650 4100
-Wire Wire Line
-	6850 5600 9650 5600
-Connection ~ 7550 5600
-Wire Wire Line
-	6200 2950 6200 4200
-Wire Wire Line
-	4150 5600 3800 5600
-Wire Wire Line
-	3800 5600 3800 3250
-Wire Wire Line
-	6600 4900 5750 4900
-Wire Wire Line
-	6350 5000 5750 5000
-Wire Wire Line
-	6100 5100 5750 5100
-Wire Wire Line
-	5750 4600 5950 4600
-Wire Wire Line
-	5950 4600 5950 4800
-Wire Wire Line
-	5950 4800 6850 4800
-Wire Wire Line
-	6850 4800 6850 5200
-Wire Wire Line
-	6950 4700 6950 5000
-Wire Wire Line
-	6200 4200 8900 4200
-Wire Wire Line
-	7550 4700 7550 4800
-Wire Wire Line
-	5750 4400 8300 4400
-Wire Wire Line
-	7550 4400 7550 4200
-Connection ~ 7550 4200
-Wire Wire Line
-	7550 4750 8150 4750
-Wire Wire Line
-	8150 4750 8150 3050
-Connection ~ 7550 4750
-Wire Wire Line
-	8900 5450 8900 5350
-Wire Wire Line
-	8900 4200 8900 4400
-Wire Wire Line
-	8900 4700 8900 4950
-Wire Wire Line
-	9400 3350 9400 4800
-Wire Wire Line
-	9400 4800 8900 4800
-Connection ~ 8900 4800
-Wire Wire Line
-	8300 4400 8300 5150
-Wire Wire Line
-	6500 4300 6500 3850
-Wire Wire Line
-	6500 3850 6650 3850
-Wire Wire Line
-	7250 4100 7250 4050
-Wire Wire Line
-	4100 2950 4100 3450
-Wire Wire Line
-	4100 3450 3800 3450
-Connection ~ 3800 3450
-Connection ~ 6200 2950
-Wire Wire Line
-	7250 3100 7250 2950
-Connection ~ 7250 2950
-Wire Wire Line
-	7250 3400 7250 3650
-Wire Wire Line
-	7900 2850 7900 3550
-Wire Wire Line
-	7900 3550 7250 3550
-Connection ~ 7250 3550
 $Comp
 L Q_NPN_CBE Q2
@@
 L Q_NPN_CBE Q1
 U 1 1 5A204BD0
-P 7450 5000
-F 0 "Q1" H 7650 5050 50  0000 L CNN
-F 1 "Q_NPN_CBE" H 7650 4950 50  0000 L CNN
-F 2 "Transistors_OldSowjetAera:OldSowjetaera_Transistor_Type-II_BigPads" H 7650 5100 50  0001 C CNN
-F 3 "" H 7450 5000 50  0001 C CNN
-	1    7450 5000
+P 7500 5100
+F 0 "Q1" H 7700 5150 50  0000 L CNN
+F 1 "Q_NPN_CBE" H 7700 5050 50  0000 L CNN
+F 2 "Transistors_OldSowjetAera:OldSowjetaera_Transistor_Type-II_BigPads" H 7700 5200 50  0001 C CNN
+F 3 "" H 7500 5100 50  0001 C CNN
+	1    7500 5100
 	1    0    0    -1
 $EndComp
@@
 $EndComp
 NoConn ~ 4150 4500
+Connection ~ 7600 5600
+Wire Wire Line
+	6850 5600 9650 5600
+Connection ~ 7600 5450
+Wire Wire Line
+	7600 5300 7600 6200
+Wire Wire Line
+	8900 5450 7600 5450
+Connection ~ 7600 5750
+Connection ~ 7600 5850
+Connection ~ 7600 5950
+Wire Wire Line
+	6950 5100 7000 5100
+Wire Wire Line
+	8150 4850 7600 4850
+Connection ~ 7600 4200
+Wire Wire Line
+	7600 4500 7600 4200
+Connection ~ 7250 3550
+Wire Wire Line
+	7900 3550 7250 3550
+Wire Wire Line
+	7900 2850 7900 3550
+Wire Wire Line
+	7250 3400 7250 3650
+Connection ~ 7250 2950
+Wire Wire Line
+	7250 3100 7250 2950
+Connection ~ 6200 2950
+Connection ~ 3800 3450
+Wire Wire Line
+	4100 3450 3800 3450
+Wire Wire Line
+	4100 2950 4100 3450
+Wire Wire Line
+	7250 4100 7250 4050
+Wire Wire Line
+	6500 3850 6650 3850
+Wire Wire Line
+	6500 4300 6500 3850
+Wire Wire Line
+	8300 4400 8300 5150
+Connection ~ 8900 4800
+Wire Wire Line
+	9400 4800 8900 4800
+Wire Wire Line
+	9400 3350 9400 4800
+Wire Wire Line
+	8900 4700 8900 4950
+Wire Wire Line
+	8900 4200 8900 4400
+Wire Wire Line
+	8900 5450 8900 5350
+Connection ~ 7600 4850
+Wire Wire Line
+	8150 3050 8150 4850
+Wire Wire Line
+	5750 4400 8300 4400
+Wire Wire Line
+	7600 4800 7600 4900
+Wire Wire Line
+	6200 4200 8900 4200
+Wire Wire Line
+	6950 4700 6950 5100
+Wire Wire Line
+	6850 4800 6850 5200
+Wire Wire Line
+	5950 4800 6850 4800
+Wire Wire Line
+	5950 4600 5950 4800
+Wire Wire Line
+	5750 4600 5950 4600
+Wire Wire Line
+	6100 5100 5750 5100
+Wire Wire Line
+	6350 5000 5750 5000
+Wire Wire Line
+	6600 4900 5750 4900
+Wire Wire Line
+	3800 3250 3800 5600
+Wire Wire Line
+	3800 5600 4150 5600
+Wire Wire Line
+	6200 2950 6200 4200
+Connection ~ 9650 4100
+Wire Wire Line
+	7250 4100 9650 4100
+Wire Wire Line
+	6500 4300 5750 4300
+Wire Wire Line
+	8400 3350 8400 3150
+Wire Wire Line
+	9400 3350 8400 3350
+Connection ~ 7600 6150
+Wire Wire Line
+	7850 6150 7850 6100
+Wire Wire Line
+	7600 6150 7850 6150
+Wire Wire Line
+	6600 5750 7600 5750
+Wire Wire Line
+	6350 5850 7600 5850
+Wire Wire Line
+	6100 5950 7600 5950
+Wire Wire Line
+	6100 4500 5750 4500
+Wire Wire Line
+	6100 4700 6100 4500
+Wire Wire Line
+	6950 4700 6100 4700
+Wire Wire Line
+	8150 3050 8850 3050
+Wire Wire Line
+	8350 2500 8350 2750
+Connection ~ 3800 2750
+Wire Wire Line
+	3500 2750 3500 2650
+Wire Wire Line
+	3800 2750 3500 2750
+Wire Wire Line
+	6350 5000 6350 5400
+Wire Wire Line
+	6100 5100 6100 5400
+Wire Wire Line
+	6600 4900 6600 5400
+Wire Wire Line
+	6100 5600 6100 5950
+Wire Wire Line
+	6350 5600 6350 5850
+Wire Wire Line
+	6600 5600 6600 5750
+Wire Wire Line
+	8350 2750 8850 2750
+Wire Wire Line
+	9650 2500 8350 2500
+Wire Wire Line
+	9650 5600 9650 2500
+Wire Wire Line
+	4100 2950 8850 2950
+Wire Wire Line
+	8400 3150 8850 3150
+Wire Wire Line
+	7900 2850 8850 2850
+Wire Wire Line
+	3800 2650 3800 2850
 $EndSCHEMATC

Commit message: Ultimos cambios
Parts:
- added J2: Conn_01x02, Pin_Headers:Pin_Header_Straight_1x02_Pitch2.54mm, symbol Conn_01x02
- U3: footprint ESP8266:NodeMCU1.0(12-E) -> lib:NodeMCU1.0(12-E)
Connections:
- net GNDPWR is gone; now on net GND: J1.1 (Pin_1), JP2.2, JP3.2, JP4.2, Q1.3 (E), Q2.3 (E), Q3.3 (E), SW2.1
- net GND: now reaches U3.10 (GND)
- net GND: now also U3.14 (GND), U3.17 (GND), U3.24 (GND), J2.1 (Pin_1)
- net +5V renamed PWR
- net PWR: now also J2.2 (Pin_2)
- no-connect marks 22 -> 18
Changed lines of the file:
@@
 F 0 "U3" H 4950 5750 60  0000 C CNN
 F 1 "NodeMCU1.0(ESP-12E)" H 4950 4050 60  0000 C CNN
-F 2 "ESP8266:NodeMCU1.0(12-E)" H 4350 4050 60  0001 C CNN
+F 2 "lib:NodeMCU1.0(12-E)" H 4350 4050 60  0001 C CNN
 F 3 "" H 4350 4050 60  0000 C CNN
 	1    4950 4900
@@
 $EndComp
 NoConn ~ 5750 4700
-NoConn ~ 5750 4800
 NoConn ~ 4150 4200
 NoConn ~ 4150 4300
@@
 NoConn ~ 5750 5300
 NoConn ~ 5750 5400
-NoConn ~ 5750 5500
 NoConn ~ 5750 5600
-NoConn ~ 4150 5500
-NoConn ~ 4150 5100
 NoConn ~ 4150 4900
 $Comp
@@
 $EndComp
 NoConn ~ 5750 4200
-$Comp
-L +5V #PWR01
-U 1 1 5A00823B
-P 3800 2650
-F 0 "#PWR01" H 3800 2500 50  0001 C CNN
-F 1 "+5V" H 3800 2790 50  0000 C CNN
-F 2 "" H 3800 2650 50  0001 C CNN
-F 3 "" H 3800 2650 50  0001 C CNN
-	1    3800 2650
-	1    0    0    -1
-$EndComp
-$Comp
-L PWR_FLAG #FLG02
-U 1 1 5A090401
-P 3500 2650
-F 0 "#FLG02" H 3500 2725 50  0001 C CNN
-F 1 "PWR_FLAG" H 3500 2800 50  0000 C CNN
-F 2 "" H 3500 2650 50  0001 C CNN
-F 3 "" H 3500 2650 50  0001 C CNN
-	1    3500 2650
-	1    0    0    -1
-$EndComp
 NoConn ~ 5750 5200
 Text Label 8600 2750 0    60   ~ 0
@@
 $EndComp
 $Comp
-L PWR_FLAG #FLG03
-U 1 1 5A09C060
-P 7850 6100
-F 0 "#FLG03" H 7850 6175 50  0001 C CNN
-F 1 "PWR_FLAG" H 7850 6250 50  0000 C CNN
-F 2 "" H 7850 6100 50  0001 C CNN
-F 3 "" H 7850 6100 50  0001 C CNN
-	1    7850 6100
-	1    0    0    -1
-$EndComp
-$Comp
 L R R1
 U 1 1 5A048190
@@
 $EndComp
 $Comp
-L GNDPWR #PWR04
-U 1 1 5A09BA2F
-P 7600 6200
-F 0 "#PWR04" H 7600 6000 50  0001 C CNN
-F 1 "GNDPWR" H 7600 6070 50  0000 C CNN
-F 2 "" H 7600 6150 50  0001 C CNN
-F 3 "" H 7600 6150 50  0001 C CNN
-	1    7600 6200
-	1    0    0    -1
-$EndComp
-$Comp
 L R R5
 U 1 1 5A0A44A8
@@
 Connection ~ 7600 5450
 Wire Wire Line
-	7600 5300 7600 6200
-Wire Wire Line
 	8900 5450 7600 5450
 Connection ~ 7600 5750
@@
 Wire Wire Line
 	9400 3350 8400 3350
-Connection ~ 7600 6150
-Wire Wire Line
-	7850 6150 7850 6100
-Wire Wire Line
-	7600 6150 7850 6150
 Wire Wire Line
 	6600 5750 7600 5750
@@
 Wire Wire Line
 	8350 2500 8350 2750
-Connection ~ 3800 2750
-Wire Wire Line
-	3500 2750 3500 2650
-Wire Wire Line
-	3800 2750 3500 2750
 Wire Wire Line
 	6350 5000 6350 5400
@@
 Wire Wire Line
 	7900 2850 8850 2850
-Wire Wire Line
-	3800 2650 3800 2850
+$Comp
+L Conn_01x02 J2
+U 1 1 5A2EF212
+P 3100 2800
+F 0 "J2" H 3100 2900 50  0000 C CNN
+F 1 "Conn_01x02" H 3100 2600 50  0000 C CNN
+F 2 "Pin_Headers:Pin_Header_Straight_1x02_Pitch2.54mm" H 3100 2800 50  0001 C CNN
+F 3 "" H 3100 2800 50  0001 C CNN
+	1    3100 2800
+	-1   0    0    1
+$EndComp
+Wire Wire Line
+	3800 2850 3800 2700
+Wire Wire Line
+	3800 2700 3300 2700
+Wire Wire Line
+	7600 5300 7600 6200
+Wire Wire Line
+	7600 6200 3300 6200
+Wire Wire Line
+	3300 6200 3300 2800
+Text Label 3400 2700 0    60   ~ 0
+PWR
+Text Label 3300 2800 0    60   ~ 0
+GND
+Wire Wire Line
+	4150 5500 3300 5500
+Connection ~ 3300 5500
+Wire Wire Line
+	5750 5500 5850 5500
+Wire Wire Line
+	5850 4800 5850 6200
+Connection ~ 5850 6200
+Wire Wire Line
+	4150 5100 3300 5100
+Connection ~ 3300 5100
+Wire Wire Line
+	5750 4800 5850 4800
+Connection ~ 5850 5500
 $EndSCHEMATC
