File: NodeMCU/matriz.sch (KiCad schematic (older format))
At the start: 17 parts, among them J1 Conn_01x05, J2 Conn_01x02, Q1 Q_NPN_CBE, Q2 Q_NPN_CBE, Q3 Q_NPN_CBE, SW1 SW_Push_Open, SW2 SW_Push, U3 NodeMCU1.0(ESP-12E)

Commit message: Pads adecuados
Parts:
- R1, R3, R5: value 500Ohm -> 10KOhm
- R2, R6: value 1000KOhm -> 10KOhm
- R4: value 1000Ohm -> 10KOhm
- U3: footprint lib:NodeMCU1.0(12-E) -> ESP8266:NodeMCU1.0(12-E)
Changed lines of the file:
@@
 F 0 "U3" H 4950 5750 60  0000 C CNN
 F 1 "NodeMCU1.0(ESP-12E)" H 4950 4050 60  0000 C CNN
-F 2 "lib:NodeMCU1.0(12-E)" H 4350 4050 60  0001 C CNN
+F 2 "ESP8266:NodeMCU1.0(12-E)" H 4350 4050 60  0001 C CNN
 F 3 "" H 4350 4050 60  0000 C CNN
 	1    4950 4900
@@
 P 7150 5100
 F 0 "R1" V 7250 5100 50  0000 C CNN
-F 1 "500Ohm" V 7350 5100 50  0000 C CNN
+F 1 "10KOhm" V 7350 5100 50  0000 C CNN
 F 2 "Resistors_THT:R_Axial_DIN0207_L6.3mm_D2.5mm_P7.62mm_Horizontal" V 7080 5100 50  0001 C CNN
 F 3 "" H 7150 5100 50  0001 C CNN
@@
 P 7600 4650
 F 0 "R2" V 7680 4650 50  0000 C CNN
-F 1 "1000KOhm" V 7750 4650 50  0000 C CNN
+F 1 "10KOhm" V 7750 4650 50  0000 C CNN
 F 2 "Resistors_THT:R_Axial_DIN0207_L6.3mm_D2.5mm_P7.62mm_Horizontal" V 7530 4650 50  0001 C CNN
 F 3 "" H 7600 4650 50  0001 C CNN
@@
 P 8450 5150
 F 0 "R3" V 8550 5150 50  0000 C CNN
-F 1 "500Ohm" V 8650 5150 50  0000 C CNN
+F 1 "10KOhm" V 8650 5150 50  0000 C CNN
 F 2 "Resistors_THT:R_Axial_DIN0207_L6.3mm_D2.5mm_P7.62mm_Horizontal" V 8380 5150 50  0001 C CNN
 F 3 "" H 8450 5150 50  0001 C CNN
@@
 P 8900 4550
 F 0 "R4" V 8980 4550 50  0000 C CNN
-F 1 "1000Ohm" V 9050 4550 50  0000 C CNN
+F 1 "10KOhm" V 9050 4550 50  0000 C CNN
 F 2 "Resistors_THT:R_Axial_DIN0207_L6.3mm_D2.5mm_P7.62mm_Horizontal" V 8830 4550 50  0001 C CNN
 F 3 "" H 8900 4550 50  0001 C CNN
@@
 P 6800 3850
 F 0 "R5" V 6900 3850 50  0000 C CNN
-F 1 "500Ohm" V 7000 3850 50  0000 C CNN
+F 1 "10KOhm" V 7000 3850 50  0000 C CNN
 F 2 "Resistors_THT:R_Axial_DIN0207_L6.3mm_D2.5mm_P7.62mm_Horizontal" V 6730 3850 50  0001 C CNN
 F 3 "" H 6800 3850 50  0001 C CNN
@@
 P 7250 3250
 F 0 "R6" V 7330 3250 50  0000 C CNN
-F 1 "1000KOhm" V 7400 3250 50  0000 C CNN
+F 1 "10KOhm" V 7400 3250 50  0000 C CNN
 F 2 "Resistors_THT:R_Axial_DIN0207_L6.3mm_D2.5mm_P7.62mm_Horizontal" V 7180 3250 50  0001 C CNN
 F 3 "" H 7250 3250 50  0001 C CNN
