File: NodeMCU/matriz.kicad_pcb (KiCad board)
At the start: 2 copper layers, 68 x 68 mm, 26 parts, among them J1 Conn_01x05, J2 Conn_01x02, Q1 Q_NPN_CBE, Q2 Q_NPN_CBE, Q3 Q_NPN_CBE, SW1 SW_Push_Open, SW2 SW_Push, U3 NodeMCU1.0(ESP-12E)

Commit message: Pads adecuados
Parts:
- added REF**: SolderWirePad_single_0-8mmDrill, Wire_Pads:SolderWirePad_single_0-8mmDrill, F.Cu at (125.7, 120.7)
- R1, R3, R5: value 500Ohm -> 10KOhm
- R2, R6: value 1000KOhm -> 10KOhm
- R4: value 1000Ohm -> 10KOhm
- moved REF** 7.82 mm to (91.4, 123.2)
- moved REF** 7.82 mm to (148.6, 123.2)
- moved GND 3.50 mm to (112.5, 77.5)
- moved U3 3.00 mm to (108.0, 106.0)
- moved GND 2.92 mm to (107.5, 77.5)
- moved GND 1.12 mm to (119.0, 77.5)
- moved JP2 1.00 mm to (104.0, 72.0)
- moved Q2 1.00 mm to (138.0, 101.0)
- moved Q3 1.00 mm to (128.0, 81.0)
- moved REF** 0.59 mm to (91.4, 72.4)
- moved JP3 0.50 mm to (110.5, 72.0)
- moved R1 0.50 mm to (124.5, 104.0)
- moved SW1 0.50 mm to (97.5, 72.0)
Routing:
- net /GND: track 199.2 -> 178.4 mm
- net Net-(JP4-Pad1): track 39.3 -> 36.1 mm
- net Net-(JP2-Pad1): track 49.0 -> 45.8 mm
- net Net-(SW2-Pad2): track 31.5 -> 28.6 mm
- net Net-(JP3-Pad1): track 42.3 -> 39.9 mm
- net Net-(Q3-Pad2): track 20.7 -> 18.3 mm
- net Net-(R1-Pad2): track 4.60 -> 6.35 mm
- net Net-(R3-Pad2): track 11.2 -> 12.5 mm
- net /PWR: track 9.92 -> 8.74 mm
- net Net-(Q2-Pad2): track 7.83 -> 6.83 mm
- net Net-(R5-Pad2): track 11.6 -> 12.5 mm
- net /V+: track 141.9 -> 141.2 mm
- net /CLK: track 87.6 -> 87.0 mm
Other:
- board size 68 x 68 mm -> 64.8 x 59.7 mm

Commit message: fix
Other:
- board size 64.8 x 59.7 mm -> 64.8 x 61.6 mm
Changed lines of the file:
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@@
     (links 40)
     (no_connects 5)
-    (area 87.252381 67.125 152.475001 127.865001)
+    (area 87.252381 67.125 152.475001 128.980001)
     (thickness 1.6)
-    (drawings 5)
+    (drawings 7)
     (tracks 122)
     (zones 0)
@@
       (effects (font (size 1 1) (thickness 0.15)))
     )
-    (pad 1 thru_hole rect (at 0 0 90) (size 2.5 1.7) (drill 1) (layers *.Cu *.Mask)
+    (pad 1 thru_hole rect (at 0 0 90) (size 2.5 1.7) (drill 0.7) (layers *.Cu *.Mask)
       (net 15 /GND))
     (pad 2 thru_hole oval (at 0 2.54 90) (size 2.5 1.7) (drill 0.7) (layers *.Cu *.Mask)
@@
       (effects (font (size 1 1) (thickness 0.15)))
     )
-    (pad 1 thru_hole circle (at 0 0) (size 1.99898 1.99898) (drill 0.8001) (layers *.Cu *.Mask)
+    (pad 1 thru_hole circle (at 0 0) (size 2 2) (drill 0.7) (layers *.Cu *.Mask)
       (net 15 /GND))
   )
@@
       (net 15 /GND))
   )
+  (gr_line (start 87.63 128.905) (end 87.63 127) (angle 90) (layer Edge.Cuts) (width 0.15))
+  (gr_line (start 152.4 128.905) (end 87.63 128.905) (angle 90) (layer Edge.Cuts) (width 0.15))
+  (gr_line (start 152.4 127) (end 152.4 128.905) (angle 90) (layer Edge.Cuts) (width 0.15))
   (gr_line (start 87.63 127) (end 87.63 67.31) (angle 90) (layer Edge.Cuts) (width 0.15))
-  (gr_line (start 152.4 127) (end 87.63 127) (angle 90) (layer Edge.Cuts) (width 0.15))
   (gr_line (start 152.4 67.31) (end 152.4 127) (angle 90) (layer Edge.Cuts) (width 0.15))
   (gr_line (start 152.4 67.31) (end 87.63 67.31) (angle 90) (layer Edge.Cuts) (width 0.15))

Commit message: esta comiendo una empanada
Parts:
- removed the GND at (129.0, 74.5)
Routing:
- net /GND: track 178.4 -> 190.0 mm
Changed lines of the file:
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@@
 (kicad_pcb (version 4) (host pcbnew 4.0.7)
   (general
-    (links 40)
-    (no_connects 5)
+    (links 39)
+    (no_connects 4)
     (area 87.252381 67.125 152.475001 128.980001)
     (thickness 1.6)
     (drawings 7)
-    (tracks 122)
+    (tracks 131)
     (zones 0)
-    (modules 27)
+    (modules 26)
     (nets 35)
   )
@@
     (mod_text_size 1 1)
     (mod_text_width 0.15)
-    (pad_size 2 2)
+    (pad_size 4.5 4.5)
     (pad_drill 0.7)
     (pad_to_mask_clearance 0.2)
@@
     (fp_circle (center 0 0) (end 2.6 0) (layer F.CrtYd) (width 0.05))
     (fp_circle (center 0 0) (end 0 -2.286) (layer F.SilkS) (width 0.12))
-    (pad 1 thru_hole circle (at 0 0) (size 4.5 4.5) (drill 4) (layers *.Cu *.Mask))
+    (pad 1 thru_hole circle (at 0 0) (size 4.5 4.5) (drill 0.7) (layers *.Cu *.Mask))
   )
   (module "lib:NodeMCU1.0(12-E)" (layer F.Cu)
@@
     (fp_circle (center 0 0) (end 2.6 0) (layer F.CrtYd) (width 0.05))
     (fp_circle (center 0 0) (end 0 -2.286) (layer F.SilkS) (width 0.12))
-    (pad 1 thru_hole circle (at 0 0) (size 4.5 4.5) (drill 4) (layers *.Cu *.Mask))
+    (pad 1 thru_hole circle (at 0 0) (size 4.5 4.5) (drill 0.7) (layers *.Cu *.Mask))
   )
   (module Connectors:1pin (layer F.Cu)
@@
     (fp_circle (center 0 0) (end 2.6 0) (layer F.CrtYd) (width 0.05))
     (fp_circle (center 0 0) (end 0 -2.286) (layer F.SilkS) (width 0.12))
-    (pad 1 thru_hole circle (at 0 0) (size 4.5 4.5) (drill 4) (layers *.Cu *.Mask))
+    (pad 1 thru_hole circle (at 0 0) (size 4.5 4.5) (drill 0.7) (layers *.Cu *.Mask))
   )
   (module Connectors:1pin (layer F.Cu)
@@
     (fp_circle (center 0 0) (end 2.6 0) (layer F.CrtYd) (width 0.05))
     (fp_circle (center 0 0) (end 0 -2.286) (layer F.SilkS) (width 0.12))
-    (pad 1 thru_hole circle (at 0 0) (size 4.5 4.5) (drill 4) (layers *.Cu *.Mask))
+    (pad 1 thru_hole circle (at 0 0) (size 4.5 4.5) (drill 0.7) (layers *.Cu *.Mask))
   )
   (module Wire_Pads:SolderWirePad_single_0-8mmDrill (layer F.Cu)
@@
   (module Wire_Pads:SolderWirePad_single_0-8mmDrill (layer F.Cu)
     (at 119 77.5)
-    (fp_text reference GND (at 0 -2.54) (layer F.SilkS)
-      (effects (font (size 1 1) (thickness 0.15)))
-    )
-    (fp_text value "" (at 0 2.54) (layer F.Fab)
-      (effects (font (size 1 1) (thickness 0.15)))
-    )
-    (pad 1 thru_hole circle (at 0 0) (size 2 2) (drill 0.7) (layers *.Cu *.Mask)
-      (net 15 /GND))
-  )
-  (module Wire_Pads:SolderWirePad_single_0-8mmDrill (layer F.Cu)
-    (at 129 74.5)
     (fp_text reference GND (at 0 -2.54) (layer F.SilkS)
       (effects (font (size 1 1) (thickness 0.15)))
@@
   (segment (start 116 106) (end 110 100) (width 1) (layer B.Cu) (net 6))
   (segment (start 110 100) (end 110 72) (width 1) (layer B.Cu) (net 6))
+  (segment (start 114 82.55) (end 114 81.58) (width 1) (layer B.Cu) (net 7))
+  (segment (start 115.951 79.629) (end 115.951 76.549) (width 1) (layer B.Cu) (net 7))
+  (segment (start 114 81.58) (end 115.951 79.629) (width 1) (layer B.Cu) (net 7))
   (segment (start 117 72) (end 117 75.5) (width 1) (layer B.Cu) (net 7))
+  (segment (start 117 75.5) (end 115.951 76.549) (width 1) (layer B.Cu) (net 7))
   (segment (start 117.46 103.46) (end 119.43 103.46) (width 1) (layer B.Cu) (net 7))
   (segment (start 114 100) (end 117.46 103.46) (width 1) (layer B.Cu) (net 7))
-  (segment (start 114 82.5) (end 114 100) (width 1) (layer B.Cu) (net 7))
-  (segment (start 115.5 81) (end 114 82.5) (width 1) (layer B.Cu) (net 7))
-  (segment (start 115.5 77) (end 115.5 81) (width 1) (layer B.Cu) (net 7))
-  (segment (start 117 75.5) (end 115.5 77) (width 1) (layer B.Cu) (net 7))
+  (segment (start 114 82.5) (end 114 82.55) (width 1) (layer B.Cu) (net 7))
+  (segment (start 114 82.55) (end 114 100) (width 1) (layer B.Cu) (net 7))
   (segment (start 119.43 93.3) (end 120.3 93.3) (width 1) (layer B.Cu) (net 8))
   (segment (start 120.3 93.3) (end 123.38 96.38) (width 1) (layer B.Cu) (net 8))
@@
   (segment (start 128 86) (end 132 86) (width 1) (layer B.Cu) (net 14))
   (segment (start 126 84) (end 128 86) (width 1) (layer B.Cu) (net 14))
+  (segment (start 132 72) (end 131.2 72) (width 1) (layer B.Cu) (net 15) (status C00000))
+  (segment (start 131.2 72) (end 122.682 80.518) (width 1) (layer B.Cu) (net 15) (status 400000))
+  (segment (start 125 88) (end 130.5 88) (width 1) (layer B.Cu) (net 15))
+  (segment (start 130.5 88) (end 139 96.5) (width 1) (layer B.Cu) (net 15))
+  (segment (start 122.682 85.682) (end 125 88) (width 1) (layer B.Cu) (net 15))
+  (segment (start 122.682 80.518) (end 122.682 85.682) (width 1) (layer B.Cu) (net 15))
+  (segment (start 112.5 77.5) (end 113.04 76.96) (width 1) (layer B.Cu) (net 15) (status C00000))
+  (segment (start 113.04 76.96) (end 112.5 77.5) (width 1) (layer B.Cu) (net 15))
+  (segment (start 130 99) (end 131.759 99) (width 1) (layer B.Cu) (net 15))
+  (segment (start 134.259 96.5) (end 139 96.5) (width 1) (layer B.Cu) (net 15))
+  (segment (start 131.759 99) (end 134.259 96.5) (width 1) (layer B.Cu) (net 15))
+  (segment (start 96.57 108.54) (end 100.5 108.54) (width 1) (layer B.Cu) (net 15))
+  (segment (start 100.33 108.585) (end 100.5 108.585) (width 1) (layer B.Cu) (net 15))
+  (segment (start 100.455 108.585) (end 100.33 108.585) (width 1) (layer B.Cu) (net 15))
+  (segment (start 100.5 108.54) (end 100.455 108.585) (width 1) (layer B.Cu) (net 15))
+  (segment (start 132 72) (end 132 76) (width 1) (layer B.Cu) (net 15))
+  (segment (start 132 76) (end 129 79) (width 1) (layer B.Cu) (net 15))
+  (segment (start 126 72) (end 132 72) (width 1) (layer B.Cu) (net 15))
+  (segment (start 139 99) (end 139 96.5) (width 1) (layer B.Cu) (net 15))
   (segment (start 121.92 116.84) (end 125.73 120.65) (width 1) (layer B.Cu) (net 15))
   (segment (start 119.43 100.92) (end 121.24 100.92) (width 1) (layer B.Cu) (net 15))
@@
   (segment (start 97.5 81) (end 92 81) (width 1) (layer B.Cu) (net 15))
   (segment (start 100.5 84) (end 97.5 81) (width 1) (layer B.Cu) (net 15))
-  (segment (start 100.5 116) (end 100.5 84) (width 1) (layer B.Cu) (net 15))
+  (segment (start 100.5 116) (end 100.5 108.585) (width 1) (layer B.Cu) (net 15))
+  (segment (start 100.5 108.585) (end 100.5 84) (width 1) (layer B.Cu) (net 15))
   (segment (start 107.5 77.5) (end 107.5 72.96) (width 1) (layer B.Cu) (net 15))
   (segment (start 107.5 72.96) (end 106.54 72) (width 1) (layer B.Cu) (net 15))
   (segment (start 113.04 72) (end 113.04 76.96) (width 1) (layer B.Cu) (net 15))
-  (segment (start 113.04 76.96) (end 112.5 77.5) (width 1) (layer B.Cu) (net 15))
   (segment (start 119.54 72) (end 119.54 76.96) (width 1) (layer B.Cu) (net 15))
   (segment (start 119.54 76.96) (end 119 77.5) (width 1) (layer B.Cu) (net 15))
-  (segment (start 129 74.5) (end 128.5 74.5) (width 1) (layer B.Cu) (net 15))
-  (segment (start 128.5 74.5) (end 123 80) (width 1) (layer B.Cu) (net 15))
-  (segment (start 139 99) (end 139 96.5) (width 1) (layer B.Cu) (net 15))
-  (segment (start 130.5 88) (end 139 96.5) (width 1) (layer B.Cu) (net 15))
-  (segment (start 125 88) (end 130.5 88) (width 1) (layer B.Cu) (net 15))
-  (segment (start 123 86) (end 125 88) (width 1) (layer B.Cu) (net 15))
-  (segment (start 123 86) (end 123 80.5) (width 1) (layer B.Cu) (net 15))
-  (segment (start 123 80) (end 123 80.5) (width 1) (layer B.Cu) (net 15))
-  (segment (start 129 74.5) (end 129 79) (width 1) (layer B.Cu) (net 15))
-  (segment (start 129 75) (end 132 72) (width 1) (layer B.Cu) (net 15))
-  (segment (start 139 99) (end 130 99) (width 1) (layer B.Cu) (net 15))
   (segment (start 130 99) (end 127.2 101.8) (width 1) (layer B.Cu) (net 15))
   (segment (start 127.2 101.8) (end 127 102) (width 1) (layer B.Cu) (net 15))
   (segment (start 127 102) (end 127 108) (width 1) (layer B.Cu) (net 15))
   (segment (start 127 108) (end 129 110) (width 1) (layer B.Cu) (net 15))
-  (segment (start 129 75) (end 126 72) (width 1) (layer B.Cu) (net 15))
   (segment (start 92 78.46) (end 92 77.5) (width 1) (layer B.Cu) (net 16))
   (segment (start 92 77.5) (end 97.5 72) (width 1) (layer B.Cu) (net 16))
