File: Slave/matriz.sch (KiCad schematic (older format))
At the start: 7 parts, among them U1 MAX7219, U2 matriz8x8, U4 interfOut

Commit message: Fix menores
Parts:
- gave numbers to parts that had none: 1
Changed lines of the file:
@@
 $EndComp
 $Comp
-L interfIn U?
+L interfIn U6
 U 1 1 5A04FCE4
 P 2050 2900
-F 0 "U?" H 2200 2500 60  0000 C CNN
+F 0 "U6" H 2200 2500 60  0000 C CNN
 F 1 "interfIn" H 2100 3200 60  0000 C CNN
 F 2 "" H 2100 3200 60  0001 C CNN

Commit message: Esquematico testeado
Parts:
- removed U2: matriz8x8, symbol matriz8x8
- removed U4: interfOut, symbol interfOut
- removed U6: interfIn, symbol interfIn
- added J1, J2: Conn_01x05, Pin_Headers:Pin_Header_Angled_1x05_Pitch2.54mm, symbol Conn_01x05
- added J3, J4: Conn_01x08, Pin_Headers:Pin_Header_Angled_1x08_Pitch2.54mm, symbol Conn_01x08
- C1: footprint (none) -> Capacitors_THT:C_Axial_L12.0mm_D6.5mm_P15.00mm_Horizontal
- CP1: footprint (none) -> Capacitors_SMD:CP_Elec_6.3x5.7
- R1: footprint (none) -> Resistors_THT:R_Axial_DIN0207_L6.3mm_D2.5mm_P7.62mm_Horizontal
- U1: footprint (none) -> Housings_DIP:DIP-24_W10.16mm_LongPads
Connections:
- net C0: now also J4.1 (Pin_1)
- net C1: now also J4.2 (Pin_2)
- net C2: now also J4.3 (Pin_3)
- net C3: now also J4.4 (Pin_4)
- net C4: now also J4.5 (Pin_5)
- net C5: now also J4.6 (Pin_6)
- net C6: now also J4.7 (Pin_7)
- net C7: now also J4.8 (Pin_8)
- net F0: now also J3.8 (Pin_8)
- net F1: now also J3.7 (Pin_7)
- net F2: now also J3.6 (Pin_6)
- net F3: now also J3.5 (Pin_5)
- net F4: now also J3.4 (Pin_4)
- net F5: now also J3.3 (Pin_3)
- net F6: now also J3.2 (Pin_2)
- net F7: now also J3.1 (Pin_1)
- net DIN: now reaches U1.1 (DIN)
- net DIN: now also J1.4 (Pin_4)
- net LD: now reaches U1.12 (LOAD)
- net LD: now also J1.1 (Pin_1), J2.5 (Pin_5)
- net CLK: now reaches U1.13 (CLK)
- net CLK: now also J1.2 (Pin_2), J2.4 (Pin_4)
- net V+: now reaches C1.1, CP1.1, R1.2, U1.19 (VCC)
- net V+: now also J1.3 (Pin_3), J2.3 (Pin_3)
- net DOUT: now reaches U1.24 (DOUT)
- net DOUT: now also J2.2 (Pin_2)
- net GND: now reaches C1.2, CP1.2, U1.4 (GND), U1.9 (GND)
- net GND: now also J1.5 (Pin_5), J2.1 (Pin_1)
Changed lines of the file:
@@
 F 0 "U1" H 6300 2400 60  0000 C CNN
 F 1 "MAX7219" H 6300 3800 60  0000 C CNN
-F 2 "" H 6900 3100 60  0000 C CNN
+F 2 "Housings_DIP:DIP-24_W10.16mm_LongPads" H 6900 3100 60  0001 C CNN
 F 3 "" H 6900 3100 60  0000 C CNN
 	1    6300 3100
@@
 F 0 "C1" H 7675 2900 50  0000 L CNN
 F 1 "0.1µF" H 7675 2700 50  0000 L CNN
-F 2 "" H 7688 2650 50  0001 C CNN
+F 2 "Capacitors_THT:C_Axial_L12.0mm_D6.5mm_P15.00mm_Horizontal" H 7688 2650 50  0001 C CNN
 F 3 "" H 7650 2800 50  0001 C CNN
 	1    7650 2800
@@
 F 0 "CP1" H 7425 2900 50  0000 L CNN
 F 1 "10µF" H 7425 2700 50  0000 L CNN
-F 2 "" H 7400 2800 50  0001 C CNN
+F 2 "Capacitors_SMD:CP_Elec_6.3x5.7" H 7400 2800 50  0001 C CNN
 F 3 "" H 7400 2800 50  0001 C CNN
 	1    7400 2800
@@
 F 0 "R1" V 7850 3050 50  0000 C TNN
 F 1 "24kOhm" V 7800 3050 50  0000 C CNN
-F 2 "" V 7930 3050 50  0001 C CNN
+F 2 "Resistors_THT:R_Axial_DIN0207_L6.3mm_D2.5mm_P7.62mm_Horizontal" V 7930 3050 50  0001 C CNN
 F 3 "" H 8000 3050 50  0001 C CNN
 	1    8000 3050
@@
 	5300 3350 5400 3250
 Entry Wire Line
-	4300 3000 4400 2900
-Entry Wire Line
-	4300 3100 4400 3000
-Entry Wire Line
-	4300 3200 4400 3100
-Entry Wire Line
-	4300 3300 4400 3200
-Entry Wire Line
-	4300 3400 4400 3300
-Entry Wire Line
-	4300 3500 4400 3400
-Entry Wire Line
-	4300 3600 4400 3500
-Entry Wire Line
-	4300 2900 4400 2800
-Text Label 4200 2900 0    47   ~ 0
+	4300 2850 4400 2750
+Entry Wire Line
+	4300 2950 4400 2850
+Entry Wire Line
+	4300 3050 4400 2950
+Entry Wire Line
+	4300 3150 4400 3050
+Entry Wire Line
+	4300 3250 4400 3150
+Entry Wire Line
+	4300 3350 4400 3250
+Entry Wire Line
+	4300 3450 4400 3350
+Entry Wire Line
+	4300 2750 4400 2650
+Text Label 4200 2750 0    47   ~ 0
 F0
-Text Label 4200 3000 0    47   ~ 0
+Text Label 4200 2850 0    47   ~ 0
 F1
-Text Label 4200 3100 0    47   ~ 0
+Text Label 4200 2950 0    47   ~ 0
 F2
-Text Label 4200 3200 0    47   ~ 0
+Text Label 4200 3050 0    47   ~ 0
 F3
-Text Label 4200 3300 0    47   ~ 0
+Text Label 4200 3150 0    47   ~ 0
 F4
-Text Label 4200 3400 0    47   ~ 0
+Text Label 4200 3250 0    47   ~ 0
 F5
-Text Label 4200 3500 0    47   ~ 0
+Text Label 4200 3350 0    47   ~ 0
 F6
-Text Label 4200 3600 0    47   ~ 0
+Text Label 4200 3450 0    47   ~ 0
 F7
 Entry Wire Line
@@
 Text Label 6950 3550 2    47   ~ 0
 F6
-$Comp
-L interfOut U4
-U 1 1 5A00A41D
-P 8800 2500
-F 0 "U4" H 8950 2100 60  0000 C CNN
-F 1 "interfOut" H 8850 2800 60  0000 C CNN
-F 2 "" H 8850 2800 60  0001 C CNN
-F 3 "" H 8850 2800 60  0001 C CNN
-	1    8800 2500
-	1    0    0    -1
-$EndComp
 Entry Wire Line
 	7000 2950 7100 2850
@@
 Entry Wire Line
 	5300 2750 5400 2650
-$Comp
-L matriz8x8 U2
-U 1 1 5A00EBC4
-P 3700 3150
-F 0 "U2" H 3900 3550 60  0000 C CNN
-F 1 "matriz8x8" H 3250 3550 60  0000 C CNN
-F 2 "" H 3900 3550 60  0001 C CNN
-F 3 "" H 3900 3550 60  0001 C CNN
-	1    3700 3150
-	1    0    0    -1
-$EndComp
-$Comp
-L interfIn U6
-U 1 1 5A04FCE4
-P 2050 2900
-F 0 "U6" H 2200 2500 60  0000 C CNN
-F 1 "interfIn" H 2100 3200 60  0000 C CNN
-F 2 "" H 2100 3200 60  0001 C CNN
-F 3 "" H 2100 3200 60  0001 C CNN
-	1    2050 2900
-	1    0    0    -1
-$EndComp
-Wire Bus Line
-	4400 2300 4400 3500
 Wire Bus Line
 	7100 2300 4400 2300
 Wire Wire Line
 	2600 2850 2600 2550
-Wire Wire Line
-	2450 2850 2600 2850
 Wire Wire Line
 	2600 2550 5700 2550
@@
 	7000 2550 6900 2550
 Wire Wire Line
-	4200 3600 4300 3600
-Wire Wire Line
-	4300 3500 4200 3500
-Wire Wire Line
-	4200 3400 4300 3400
-Wire Wire Line
-	4300 3300 4200 3300
-Wire Wire Line
-	4200 3200 4300 3200
-Wire Wire Line
-	4300 3100 4200 3100
-Wire Wire Line
-	4200 3000 4300 3000
-Wire Wire Line
-	4300 2900 4200 2900
+	4200 3450 4300 3450
+Wire Wire Line
+	4300 3350 4200 3350
+Wire Wire Line
+	4200 3250 4300 3250
+Wire Wire Line
+	4300 3150 4200 3150
+Wire Wire Line
+	4200 3050 4300 3050
+Wire Wire Line
+	4300 2950 4200 2950
+Wire Wire Line
+	4200 2850 4300 2850
+Wire Wire Line
+	4300 2750 4200 2750
 Wire Wire Line
 	5700 3650 5700 4400
@@
 	7950 2350 8500 2350
 Wire Wire Line
-	2500 2200 2500 2750
-Wire Wire Line
-	2500 2750 2450 2750
-Wire Wire Line
 	7650 2650 7650 2200
 Connection ~ 7650 2200
@@
 Wire Wire Line
 	2800 4400 2800 3150
-Wire Wire Line
-	2800 3150 2450 3150
 Connection ~ 5700 3900
 Wire Wire Line
@@
 Wire Wire Line
 	2850 2050 2850 2950
-Wire Wire Line
-	2850 2950 2450 2950
 Connection ~ 8150 2550
-Wire Wire Line
-	2450 3050 2600 3050
 Wire Wire Line
 	2600 3050 2600 4550
@@
 	7150 4550 7150 3650
 Connection ~ 7150 3650
+$Comp
+L Conn_01x05 J1
+U 1 1 5A09A051
+P 1850 2950
+F 0 "J1" H 1850 3250 50  0000 C CNN
+F 1 "Conn_01x05" H 1850 2650 50  0000 C CNN
+F 2 "Pin_Headers:Pin_Header_Angled_1x05_Pitch2.54mm" H 1850 2950 50  0001 C CNN
+F 3 "" H 1850 2950 50  0001 C CNN
+	1    1850 2950
+	-1   0    0    1
+$EndComp
+$Comp
+L Conn_01x05 J2
+U 1 1 5A09A094
+P 8700 2550
+F 0 "J2" H 8700 2850 50  0000 C CNN
+F 1 "Conn_01x05" H 8700 2250 50  0000 C CNN
+F 2 "Pin_Headers:Pin_Header_Angled_1x05_Pitch2.54mm" H 8700 2550 50  0001 C CNN
+F 3 "" H 8700 2550 50  0001 C CNN
+	1    8700 2550
+	1    0    0    -1
+$EndComp
+Text Label 2100 2750 0    60   ~ 0
+GND
+Text Label 2100 2850 0    60   ~ 0
+DIN
+Text Label 2100 2950 0    60   ~ 0
+V+
+Text Label 2100 3050 0    60   ~ 0
+CLK
+Text Label 2100 3150 0    60   ~ 0
+LD
+Wire Wire Line
+	2800 3150 2050 3150
+Wire Wire Line
+	2050 3050 2600 3050
+Wire Wire Line
+	2850 2950 2050 2950
+Wire Wire Line
+	2050 2850 2600 2850
+Wire Wire Line
+	2500 2750 2500 2200
+Wire Wire Line
+	2050 2750 2500 2750
+Text Label 8450 2350 2    60   ~ 0
+GND
+Text Label 8450 2450 2    60   ~ 0
+DOUT
+Text Label 8450 2550 2    60   ~ 0
+V+
+Text Label 8450 2650 2    60   ~ 0
+CLK
+Text Label 8450 2750 2    60   ~ 0
+LD
+$Comp
+L Conn_01x08 J3
+U 1 1 5A09A91B
+P 4000 3150
+F 0 "J3" H 4000 3550 50  0000 C CNN
+F 1 "Conn_01x08" H 4000 2650 50  0000 C CNN
+F 2 "Pin_Headers:Pin_Header_Angled_1x08_Pitch2.54mm" H 4000 3150 50  0001 C CNN
+F 3 "" H 4000 3150 50  0001 C CNN
+	1    4000 3150
+	-1   0    0    1
+$EndComp
+$Comp
+L Conn_01x08 J4
+U 1 1 5A09A95A
+P 3400 3800
+F 0 "J4" H 3400 4200 50  0000 C CNN
+F 1 "Conn_01x08" H 3400 3300 50  0000 C CNN
+F 2 "Pin_Headers:Pin_Header_Angled_1x08_Pitch2.54mm" H 3400 3800 50  0001 C CNN
+F 3 "" H 3400 3800 50  0001 C CNN
+	1    3400 3800
+	0    -1   -1   0
+$EndComp
+Wire Bus Line
+	4400 2300 4400 3350
 $EndSCHEMATC

Commit message: Footprint slave
Parts:
- C1: footprint Capacitors_THT:C_Axial_L12.0mm_D6.5mm_P15.00mm_Horizontal -> Capacitors_THT:C_Axial_L3.8mm_D2.6mm_P7.50mm_Horizontal
Other:
- moved on the sheet: J1, J3, J4

Commit message: Pistas todas de 1mm, limite y unidades mecanicas
Parts:
- CP1: footprint Capacitors_SMD:CP_Elec_6.3x5.7 -> Capacitors_THT:CP_Radial_Tantal_D8.0mm_P5.00mm
- J1, J2: footprint Pin_Headers:Pin_Header_Angled_1x05_Pitch2.54mm -> Pin_Headers:Pin_Header_Straight_1x05_Pitch2.54mm
- J3, J4: footprint Pin_Headers:Pin_Header_Angled_1x08_Pitch2.54mm -> Pin_Headers:Pin_Header_Straight_1x08_Pitch2.54mm
Changed lines of the file:
@@
 F 0 "CP1" H 7425 2900 50  0000 L CNN
 F 1 "10µF" H 7425 2700 50  0000 L CNN
-F 2 "Capacitors_SMD:CP_Elec_6.3x5.7" H 7400 2800 50  0001 C CNN
+F 2 "Capacitors_THT:CP_Radial_Tantal_D8.0mm_P5.00mm" H 7400 2800 50  0001 C CNN
 F 3 "" H 7400 2800 50  0001 C CNN
 	1    7400 2800
@@
 F 0 "J1" H 2800 3250 50  0000 C CNN
 F 1 "Conn_01x05" H 2800 2650 50  0000 C CNN
-F 2 "Pin_Headers:Pin_Header_Angled_1x05_Pitch2.54mm" H 2800 2950 50  0001 C CNN
+F 2 "Pin_Headers:Pin_Header_Straight_1x05_Pitch2.54mm" H 2800 2950 50  0001 C CNN
 F 3 "" H 2800 2950 50  0001 C CNN
 	1    2800 2950
@@
 F 0 "J2" H 8700 2850 50  0000 C CNN
 F 1 "Conn_01x05" H 8700 2250 50  0000 C CNN
-F 2 "Pin_Headers:Pin_Header_Angled_1x05_Pitch2.54mm" H 8700 2550 50  0001 C CNN
+F 2 "Pin_Headers:Pin_Header_Straight_1x05_Pitch2.54mm" H 8700 2550 50  0001 C CNN
 F 3 "" H 8700 2550 50  0001 C CNN
 	1    8700 2550
@@
 F 0 "J3" H 4600 3550 50  0000 C CNN
 F 1 "Conn_01x08" H 4600 2650 50  0000 C CNN
-F 2 "Pin_Headers:Pin_Header_Angled_1x08_Pitch2.54mm" H 4600 3150 50  0001 C CNN
+F 2 "Pin_Headers:Pin_Header_Straight_1x08_Pitch2.54mm" H 4600 3150 50  0001 C CNN
 F 3 "" H 4600 3150 50  0001 C CNN
 	1    4600 3150
@@
 F 0 "J4" H 4300 4200 50  0000 C CNN
 F 1 "Conn_01x08" H 4300 3300 50  0000 C CNN
-F 2 "Pin_Headers:Pin_Header_Angled_1x08_Pitch2.54mm" H 4300 3800 50  0001 C CNN
+F 2 "Pin_Headers:Pin_Header_Straight_1x08_Pitch2.54mm" H 4300 3800 50  0001 C CNN
 F 3 "" H 4300 3800 50  0001 C CNN
 	1    4300 3800

Commit message: Ultimos cambios
Parts:
- U1: footprint Housings_DIP:DIP-24_W10.16mm_LongPads -> Housings_DIP:DIP-24_W7.62mm_LongPads
Changed lines of the file:
@@
 F 0 "U1" H 6300 2400 60  0000 C CNN
 F 1 "MAX7219" H 6300 3800 60  0000 C CNN
-F 2 "Housings_DIP:DIP-24_W10.16mm_LongPads" H 6900 3100 60  0001 C CNN
+F 2 "Housings_DIP:DIP-24_W7.62mm_LongPads" H 6900 3100 60  0001 C CNN
 F 3 "" H 6900 3100 60  0000 C CNN
 	1    6300 3100
